File: Hardware/Freya-sensor.kicad_sch (KiCad schematic)
At the start: 17 parts, among them J1 JST4.0, Q1 BS170, Q2 BS170, U1 BME680, U2 VEML6030, U3 MIC5225-3.3YM5, U4 AS7331

Commit message: Electronics v2.1
Parts:
- J1: value JST4.0 -> HY2.0-4P
Other:
- note added: "1.2"
- note added: "Copyright© 2026 Sanne 'SpuQ' Santens"
- note added: "Freya Terra Sensor"
- note added: "Rev.: 1.2 License: CERN-OHL-W"
- note added: "https://github.com/Freya-Vivariums"
- note removed: "1.0"
- note removed: "Freya - Vivarium Control System"
- note removed: "Sensor Rev.: 1.1 by Sanne 'SpuQ' Santens, early 2026"
