File: Hardware/Freya-sensor.kicad_pcb (KiCad board)
At the start: 2 copper layers, 50 x 15 mm, 23 parts, among them J1 Grove, Q1 BS170, Q2 BS170, U1 BME680, U2 VEML6030, U3 MIC5225-3.3YM5, U4 AS7331

Commit message: Electronics v2.1
Other:
- board text added: "Freya Terra Sensor"
- board text added: "Rev.: 1.2 License: CERN-OHL-W Copyright© 2026 Sanne 'SpuQ' Santens https://github.com/Freya-Vivariums"
- board text added: "TERRA SENSOR V1.2"
- board text removed: "Freya - Vivarium Control System"
- board text removed: "SENSOR Rev. 1.1"
- board text removed: "Sensor Rev.: 1.1 by Sanne 'SpuQ' Santens, early 2026"

Commit message: Hardware: pre manufacturing
Parts:
- J1: value Grove -> HY2.0-4P
Changed lines of the file:
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@@
 		(filling no)
 		(pcbplotparams
-			(layerselection 0x00000000_00000000_5555555d_55555550)
-			(plot_on_all_layers_selection 0x00000000_00000000_00000080_02000000)
+			(layerselection 0x00000000_00000000_55555555_5755f5ff)
+			(plot_on_all_layers_selection 0x00000000_00000000_00000000_02000000)
 			(disableapertmacros no)
 			(usegerberextensions no)
@@
 			(dashed_line_gap_ratio 3)
 			(svgprecision 4)
-			(plotframeref yes)
+			(plotframeref no)
 			(mode 1)
 			(useauxorigin yes)
@@
 			(crossoutdnponfab yes)
 			(subtractmaskfromsilk no)
-			(outputformat 4)
+			(outputformat 1)
 			(mirror no)
 			(drillshape 0)
@@
 	)
 	(footprint ""
+		(locked yes)
 		(layer "F.Cu")
 		(at 165.9 101.4)
@@
 			(at 0 0 0)
 			(layer "F.SilkS")
+			(hide yes)
 			(effects
 				(font
@@
 			)
 		)
+		(attr board_only exclude_from_pos_files exclude_from_bom)
 		(duplicate_pad_numbers_are_jumpers no)
 		(pad "" smd circle
@@
 	)
 	(footprint "Fiducial:Fiducial_0.5mm_Mask1.5mm"
+		(locked yes)
 		(layer "F.Cu")
 		(at 141.4 101.4)
@@
 			)
 		)
-		(attr smd)
+		(attr smd board_only exclude_from_pos_files exclude_from_bom)
 		(duplicate_pad_numbers_are_jumpers no)
 		(fp_circle
@@
 	)
 	(footprint ""
+		(locked yes)
 		(layer "F.Cu")
 		(at 141.4 113.6)
@@
 			(at 0 0 0)
 			(layer "F.SilkS")
+			(hide yes)
 			(effects
 				(font
@@
 			)
 		)
+		(attr board_only exclude_from_pos_files exclude_from_bom)
 		(duplicate_pad_numbers_are_jumpers no)
 		(pad "" smd circle
@@
 	)
 	(footprint "emcosys:Grove_SMD_right_angle"
+		(locked yes)
 		(layer "F.Cu")
 		(at 188.5 107.5)
@@
 			)
 		)
-		(property "Value" "Grove"
+		(property "Value" "HY2.0-4P"
 			(at -1.65 0 90)
 			(unlocked yes)
@@
 		)
 		(model "/home/tom/Projects/Freya-Edgeberry/Freya-terra-sensor/Documentation/Enclosure.wrl"
+			(hide yes)
 			(offset
 				(xyz -126 0 0)
